File: breakout-bitsy/Revision A1/caravel-breakout-bitsy-RevA1.kicad_sch (KiCad schematic)
At the start: 14 parts, among them CON1 REF-182665-01, CON2 REF-182665-01, CON3 73251-1352, U1 Caravel, U2 TLV73318PDBV

Commit message: WIP checkin for comments
Parts:
- removed C1, C2, C3, C4, C5, C6, C7: 0.1uf, Capacitor_SMD:C_0402_1005Metric, symbol Device:C
- removed C8, C9: 0.1uf, Capacitor_SMD:C_0603_1608Metric, symbol Device:C
- removed CON3: 73251-1352, ok-connectors:TE_5-1814832-2, symbol ok-connectors:SMA_TH
- removed U1: Caravel, ok-chips:Caravel_WLCSP, symbol ok-chips:Caravel_WLCSP
- removed U2: TLV73318PDBV, Package_TO_SOT_SMD:SOT-23-5, symbol Regulator_Linear:TLV73318PDBV
- added A1: iCEBreaker_Bitsy, ok-modules:iCEBreaker_Bitsy_THT, symbol ok-modules:iCEBreaker_Bitsy
- CON1, CON2: value REF-182665-01 -> 2x20 2.54mm Socket; footprint ok-connectors:REF-182665-01 -> ok-connectors:PinSocket_2x20_P2.54mm_Vertical_Center_Rev
