File: breakout-wlcsp/Revision A1/caravel-breakout-wlcsp-RevA1.kicad_sch (KiCad schematic)
At the start: 14 parts, among them CON1 REF-182665-01, CON2 REF-182665-01, CON3 73251-1352, U1 Caravel, U2 TLV73318PDBV

Commit message: initial check-in for RevA1
Parts:
- removed C8, C9: 0.1uf, Capacitor_SMD:C_0603_1608Metric, symbol Device:C
- removed U2: TLV73318PDBV, Package_TO_SOT_SMD:SOT-23-5, symbol Regulator_Linear:TLV73318PDBV
Other:
- moved on the sheet: CON3
Changed lines of the file:
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@@
   (junction (at 41.91 93.98) (diameter 0) (color 0 0 0 0)
   )
-  (junction (at 111.76 176.53) (diameter 0) (color 0 0 0 0)
+  (junction (at 111.125 176.53) (diameter 0) (color 0 0 0 0)
   )
   (junction (at 212.09 62.23) (diameter 0) (color 0 0 0 0)
@@
   (junction (at 100.33 130.81) (diameter 0) (color 0 0 0 0)
   )
-  (junction (at 111.76 179.07) (diameter 0) (color 0 0 0 0)
+  (junction (at 111.125 179.07) (diameter 0) (color 0 0 0 0)
   )
   (junction (at 234.95 62.23) (diameter 0) (color 0 0 0 0)
@@
   (junction (at 162.56 93.98) (diameter 0) (color 0 0 0 0)
   )
-  (junction (at 111.76 173.99) (diameter 0) (color 0 0 0 0)
+  (junction (at 111.125 173.99) (diameter 0) (color 0 0 0 0)
   )
   (junction (at 212.09 128.27) (diameter 0) (color 0 0 0 0)
@@
     (stroke (width 0) (type default) (color 0 0 0 0))
   )
-  (wire (pts (xy 109.22 176.53) (xy 111.76 176.53))
+  (wire (pts (xy 108.585 176.53) (xy 111.125 176.53))
     (stroke (width 0) (type default) (color 0 0 0 0))
   )
@@
     (stroke (width 0) (type default) (color 0 0 0 0))
   )
-  (wire (pts (xy 111.76 173.99) (xy 111.76 176.53))
+  (wire (pts (xy 111.125 173.99) (xy 111.125 176.53))
     (stroke (width 0) (type default) (color 0 0 0 0))
   )
@@
     (stroke (width 0) (type default) (color 0 0 0 0))
   )
-  (wire (pts (xy 83.82 175.26) (xy 88.9 175.26))
+  (wire (pts (xy 83.185 175.26) (xy 88.265 175.26))
     (stroke (width 0) (type default) (color 0 0 0 0))
   )
@@
     (stroke (width 0) (type default) (color 0 0 0 0))
   )
-  (wire (pts (xy 111.76 179.07) (xy 111.76 181.61))
-    (stroke (width 0) (type default) (color 0 0 0 0))
-  )
-  (wire (pts (xy 111.76 176.53) (xy 111.76 179.07))
+  (wire (pts (xy 111.125 179.07) (xy 111.125 181.61))
+    (stroke (width 0) (type default) (color 0 0 0 0))
+  )
+  (wire (pts (xy 111.125 176.53) (xy 111.125 179.07))
     (stroke (width 0) (type default) (color 0 0 0 0))
   )
@@
     (stroke (width 0) (type default) (color 0 0 0 0))
   )
-  (wire (pts (xy 109.22 173.99) (xy 111.76 173.99))
+  (wire (pts (xy 108.585 173.99) (xy 111.125 173.99))
     (stroke (width 0) (type default) (color 0 0 0 0))
   )
@@
     (stroke (width 0) (type default) (color 0 0 0 0))
   )
-  (wire (pts (xy 109.22 171.45) (xy 111.76 171.45))
+  (wire (pts (xy 108.585 171.45) (xy 111.125 171.45))
     (stroke (width 0) (type default) (color 0 0 0 0))
   )
@@
     (stroke (width 0) (type default) (color 0 0 0 0))
   )
-  (wire (pts (xy 109.22 179.07) (xy 111.76 179.07))
+  (wire (pts (xy 108.585 179.07) (xy 111.125 179.07))
     (stroke (width 0) (type default) (color 0 0 0 0))
   )
@@
     (stroke (width 0) (type default) (color 0 0 0 0))
   )
-  (wire (pts (xy 111.76 171.45) (xy 111.76 173.99))
+  (wire (pts (xy 111.125 171.45) (xy 111.125 173.99))
     (stroke (width 0) (type default) (color 0 0 0 0))
   )
@@
     )
   )
-  (global_label "xclk" (shape input) (at 83.82 175.26 180) (fields_autoplaced)
-    (effects (font (size 1.27 1.27)) (justify right))
-    (property "Intersheet References" "${INTERSHEET_REFS}" (id 0) (at -143.51 36.83 0)
+  (global_label "xclk" (shape input) (at 83.185 175.26 180) (fields_autoplaced)
+    (effects (font (size 1.27 1.27)) (justify right))
+    (property "Intersheet References" "${INTERSHEET_REFS}" (id 0) (at -144.145 36.83 0)
       (effects (font (size 1.27 1.27)) hide)
     )
@@
     (pin "1")
   )
-  (symbol (lib_id "Regulator_Linear:TLV73318PDBV") (at 144.78 157.48 0) (unit 1)
-    (in_bom yes) (on_board yes) (fields_autoplaced)
-    (property "Reference" "U2" (id 0) (at 144.78 147.32 0))
-    (property "Value" "TLV73318PDBV" (id 1) (at 144.78 149.86 0))
-    (property "Footprint" "Package_TO_SOT_SMD:SOT-23-5" (id 2) (at 144.78 149.225 0)
-      (effects (font (size 1.27 1.27) italic) hide)
-    )
-    (property "Datasheet" "http://www.ti.com/lit/ds/symlink/tlv733p.pdf" (id 3) (at 144.78 157.48 0)
-      (effects (font (size 1.27 1.27)) hide)
-    )
-    (pin "1")
-    (pin "2")
-    (pin "3")
-    (pin "4")
-    (pin "5")
-  )
   (symbol (lib_id "Connector_Generic:Conn_02x20_Odd_Even") (at 222.25 52.07 0) (unit 1)
     (in_bom yes) (on_board yes)
@@
     (pin "1")
   )
-  (symbol (lib_id "Device:C") (at 129.54 158.75 180) (unit 1)
-    (in_bom yes) (on_board yes)
-    (property "Reference" "C8" (id 0) (at 125.73 158.75 90))
-    (property "Value" "0.1uf" (id 1) (at 123.19 158.75 90))
-    (property "Footprint" "Capacitor_SMD:C_0603_1608Metric" (id 2) (at 128.5748 154.94 0)
-      (effects (font (size 1.27 1.27)) hide)
-    )
-    (property "Datasheet" "~" (id 3) (at 129.54 158.75 0)
-      (effects (font (size 1.27 1.27)) hide)
-    )
-    (pin "1")
-    (pin "2")
-  )
   (symbol (lib_id "power:GND") (at 212.09 154.94 0) (unit 1)
     (in_bom yes) (on_board yes)
@@
     (pin "1")
   )
-  (symbol (lib_id "power:GND") (at 111.76 181.61 0) (unit 1)
-    (in_bom yes) (on_board yes)
-    (property "Reference" "#PWR0101" (id 0) (at 111.76 187.96 0)
-      (effects (font (size 1.27 1.27)) hide)
-    )
-    (property "Value" "GND" (id 1) (at 111.76 186.69 90))
-    (property "Footprint" "" (id 2) (at 111.76 181.61 0)
-      (effects (font (size 1.27 1.27)) hide)
-    )
-    (property "Datasheet" "" (id 3) (at 111.76 181.61 0)
-      (effects (font (size 1.27 1.27)) hide)
-    )
-    (pin "1")
-  )
-  (symbol (lib_id "Device:C") (at 160.02 158.75 180) (unit 1)
-    (in_bom yes) (on_board yes)
-    (property "Reference" "C9" (id 0) (at 156.21 158.75 90))
-    (property "Value" "0.1uf" (id 1) (at 153.67 158.75 90))
-    (property "Footprint" "Capacitor_SMD:C_0603_1608Metric" (id 2) (at 159.0548 154.94 0)
-      (effects (font (size 1.27 1.27)) hide)
-    )
-    (property "Datasheet" "~" (id 3) (at 160.02 158.75 0)
-      (effects (font (size 1.27 1.27)) hide)
-    )
-    (pin "1")
-    (pin "2")
+  (symbol (lib_id "power:GND") (at 111.125 181.61 0) (unit 1)
+    (in_bom yes) (on_board yes)
+    (property "Reference" "#PWR0101" (id 0) (at 111.125 187.96 0)
+      (effects (font (size 1.27 1.27)) hide)
+    )
+    (property "Value" "GND" (id 1) (at 111.125 186.69 90))
+    (property "Footprint" "" (id 2) (at 111.125 181.61 0)
+      (effects (font (size 1.27 1.27)) hide)
+    )
+    (property "Datasheet" "" (id 3) (at 111.125 181.61 0)
+      (effects (font (size 1.27 1.27)) hide)
+    )
+    (pin "1")
   )
   (symbol (lib_id "power:GND") (at 234.95 154.94 0) (unit 1)
@@
     (pin "9")
   )
-  (symbol (lib_id "ok-connectors:SMA_TH") (at 99.06 175.26 0) (unit 1)
-    (in_bom yes) (on_board yes)
-    (property "Reference" "CON3" (id 0) (at 93.98 168.91 0))
-    (property "Value" "73251-1352" (id 1) (at 97.79 181.61 0))
-    (property "Footprint" "ok-connectors:TE_5-1814832-2" (id 2) (at 91.44 182.88 0)
-      (effects (font (size 1.27 1.27)) (justify left) hide)
-    )
-    (property "Datasheet" "" (id 3) (at 99.06 175.26 0)
+  (symbol (lib_id "ok-connectors:SMA_TH") (at 98.425 175.26 0) (unit 1)
+    (in_bom yes) (on_board yes)
+    (property "Reference" "CON3" (id 0) (at 93.345 168.91 0))
+    (property "Value" "73251-1352" (id 1) (at 97.155 181.61 0))
+    (property "Footprint" "ok-connectors:TE_5-1814832-2" (id 2) (at 90.805 182.88 0)
+      (effects (font (size 1.27 1.27)) (justify left) hide)
+    )
+    (property "Datasheet" "" (id 3) (at 98.425 175.26 0)
       (effects (font (size 1.27 1.27)) hide)
     )
@@
       (reference "C7") (unit 1) (value "0.1uf") (footprint "Capacitor_SMD:C_0402_1005Metric")
     )
-    (path "/748e673c-62ba-48f2-8c93-fcf00774af87"
-      (reference "C8") (unit 1) (value "0.1uf") (footprint "Capacitor_SMD:C_0603_1608Metric")
-    )
-    (path "/9c14b6d3-b2f0-4fdc-9232-d4338971c346"
-      (reference "C9") (unit 1) (value "0.1uf") (footprint "Capacitor_SMD:C_0603_1608Metric")
-    )
     (path "/3e1c8ec7-6848-47a8-83de-e92b32eb31d7"
       (reference "CON1") (unit 1) (value "REF-182665-01") (footprint "ok-connectors:REF-182665-01")
@@
       (reference "U1") (unit 1) (value "Caravel") (footprint "ok-chips:Caravel_WLCSP")
     )
-    (path "/0d29bb03-4b1f-4213-ba3c-74ea953f1fc4"
-      (reference "U2") (unit 1) (value "TLV73318PDBV") (footprint "Package_TO_SOT_SMD:SOT-23-5")
-    )
-  )
+  )
