File: breakout-wlcsp/caravel-breakout-wlcsp.kicad_sch (KiCad schematic)
At the start: 11 parts, among them CON1 REF-182665-01, CON2 REF-182665-01, CON3 73251-1352, U1 Caravel

Commit message: Revision A2 release and re-org
Other:
- note added: "Caravel breakout (WLCSP package)"
- title: (none) -> Caravel breakout (WLCSP package)
Changed lines of the file:
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@@
 (kicad_sch (version 20230121) (generator eeschema)
   (paper "A")
+  (title_block
+    (title "Caravel breakout (WLCSP package)")
+    (date "2023-06-20")
+    (rev "A2")
+  )
   (junction (at 41.91 93.98) (diameter 0) (color 0 0 0 0)
   )
@@
   (wire (pts (xy 142.24 60.96) (xy 138.43 60.96))
     (stroke (width 0) (type default))
+  )
+  (text "Caravel breakout (WLCSP package)" (at 118.11 20.32 0)
+    (effects (font (size 3 3) (thickness 0.6) bold) (justify left bottom))
   )
   (global_label "mprj_io[11]" (shape input) (at 207.01 107.95 180) (fields_autoplaced)
@@
     (pin "F9")
     (instances
-      (project "caravel-breakout-wlcsp-RevA1"
+      (project "caravel-breakout-wlcsp"
         (path "/b38c65ac-2d57-46f9-9a32-ad09573ee400"
           (reference "U1") (unit 1)
@@
     (pin "2")
     (instances
-      (project "caravel-breakout-wlcsp-RevA1"
+      (project "caravel-breakout-wlcsp"
         (path "/b38c65ac-2d57-46f9-9a32-ad09573ee400"
           (reference "C3") (unit 1)
@@
     (pin "1")
     (instances
-      (project "caravel-breakout-wlcsp-RevA1"
+      (project "caravel-breakout-wlcsp"
         (path "/b38c65ac-2d57-46f9-9a32-ad09573ee400"
           (reference "#PWR013") (unit 1)
@@
     (pin "1")
     (instances
-      (project "caravel-breakout-wlcsp-RevA1"
+      (project "caravel-breakout-wlcsp"
         (path "/b38c65ac-2d57-46f9-9a32-ad09573ee400"
           (reference "#PWR023") (unit 1)
@@
     (pin "1")
     (instances
-      (project "caravel-breakout-wlcsp-RevA1"
+      (project "caravel-breakout-wlcsp"
         (path "/b38c65ac-2d57-46f9-9a32-ad09573ee400"
           (reference "#PWR021") (unit 1)
@@
     (pin "1")
     (instances
-      (project "caravel-breakout-wlcsp-RevA1"
+      (project "caravel-breakout-wlcsp"
         (path "/b38c65ac-2d57-46f9-9a32-ad09573ee400"
           (reference "#PWR022") (unit 1)
@@
     (pin "1")
     (instances
-      (project "caravel-breakout-wlcsp-RevA1"
+      (project "caravel-breakout-wlcsp"
         (path "/b38c65ac-2d57-46f9-9a32-ad09573ee400"
           (reference "#PWR012") (unit 1)
@@
     (pin "1")
     (instances
-      (project "caravel-breakout-wlcsp-RevA1"
+      (project "caravel-breakout-wlcsp"
         (path "/b38c65ac-2d57-46f9-9a32-ad09573ee400"
           (reference "#PWR014") (unit 1)
@@
     (pin "1")
     (instances
-      (project "caravel-breakout-wlcsp-RevA1"
+      (project "caravel-breakout-wlcsp"
         (path "/b38c65ac-2d57-46f9-9a32-ad09573ee400"
           (reference "#PWR011") (unit 1)
@@
     (pin "1")
     (instances
-      (project "caravel-breakout-wlcsp-RevA1"
+      (project "caravel-breakout-wlcsp"
         (path "/b38c65ac-2d57-46f9-9a32-ad09573ee400"
           (reference "#PWR07") (unit 1)
@@
     (pin "2")
     (instances
-      (project "caravel-breakout-wlcsp-RevA1"
+      (project "caravel-breakout-wlcsp"
         (path "/b38c65ac-2d57-46f9-9a32-ad09573ee400"
           (reference "C6") (unit 1)
@@
     (pin "2")
     (instances
-      (project "caravel-breakout-wlcsp-RevA1"
+      (project "caravel-breakout-wlcsp"
         (path "/b38c65ac-2d57-46f9-9a32-ad09573ee400"
           (reference "C4") (unit 1)
@@
     (pin "1")
     (instances
-      (project "caravel-breakout-wlcsp-RevA1"
+      (project "caravel-breakout-wlcsp"
         (path "/b38c65ac-2d57-46f9-9a32-ad09573ee400"
           (reference "#PWR027") (unit 1)
@@
     (pin "1")
     (instances
-      (project "caravel-breakout-wlcsp-RevA1"
+      (project "caravel-breakout-wlcsp"
         (path "/b38c65ac-2d57-46f9-9a32-ad09573ee400"
           (reference "#PWR026") (unit 1)
@@
     (pin "1")
     (instances
-      (project "caravel-breakout-wlcsp-RevA1"
+      (project "caravel-breakout-wlcsp"
         (path "/b38c65ac-2d57-46f9-9a32-ad09573ee400"
           (reference "#PWR05") (unit 1)
@@
     (pin "2")
     (instances
-      (project "caravel-breakout-wlcsp-RevA1"
+      (project "caravel-breakout-wlcsp"
         (path "/b38c65ac-2d57-46f9-9a32-ad09573ee400"
           (reference "C2") (unit 1)
@@
     (pin "1")
     (instances
-      (project "caravel-breakout-wlcsp-RevA1"
+      (project "caravel-breakout-wlcsp"
         (path "/b38c65ac-2d57-46f9-9a32-ad09573ee400"
           (reference "#PWR017") (unit 1)
@@
     (pin "2")
     (instances
-      (project "caravel-breakout-wlcsp-RevA1"
+      (project "caravel-breakout-wlcsp"
         (path "/b38c65ac-2d57-46f9-9a32-ad09573ee400"
           (reference "C7") (unit 1)
@@
     (pin "2")
     (instances
-      (project "caravel-breakout-wlcsp-RevA1"
+      (project "caravel-breakout-wlcsp"
         (path "/b38c65ac-2d57-46f9-9a32-ad09573ee400"
           (reference "C5") (unit 1)
@@
     (pin "1")
     (instances
-      (project "caravel-breakout-wlcsp-RevA1"
+      (project "caravel-breakout-wlcsp"
         (path "/b38c65ac-2d57-46f9-9a32-ad09573ee400"
           (reference "#PWR016") (unit 1)
@@
     (pin "2")
     (instances
-      (project "caravel-breakout-wlcsp-RevA1"
+      (project "caravel-breakout-wlcsp"
         (path "/b38c65ac-2d57-46f9-9a32-ad09573ee400"
           (reference "C1") (unit 1)
@@
     (pin "1")
     (instances
-      (project "caravel-breakout-wlcsp-RevA1"
+      (project "caravel-breakout-wlcsp"
         (path "/b38c65ac-2d57-46f9-9a32-ad09573ee400"
           (reference "#PWR09") (unit 1)
@@
     (pin "9")
     (instances
-      (project "caravel-breakout-wlcsp-RevA1"
+      (project "caravel-breakout-wlcsp"
         (path "/b38c65ac-2d57-46f9-9a32-ad09573ee400"
           (reference "CON1") (unit 1)
@@
     (pin "1")
     (instances
-      (project "caravel-breakout-wlcsp-RevA1"
+      (project "caravel-breakout-wlcsp"
         (path "/b38c65ac-2d57-46f9-9a32-ad09573ee400"
           (reference "#PWR0104") (unit 1)
@@
     (pin "1")
     (instances
-      (project "caravel-breakout-wlcsp-RevA1"
+      (project "caravel-breakout-wlcsp"
         (path "/b38c65ac-2d57-46f9-9a32-ad09573ee400"
           (reference "#PWR0105") (unit 1)
@@
     (pin "1")
     (instances
-      (project "caravel-breakout-wlcsp-RevA1"
+      (project "caravel-breakout-wlcsp"
         (path "/b38c65ac-2d57-46f9-9a32-ad09573ee400"
           (reference "#PWR0102") (unit 1)
@@
     (pin "1")
     (instances
-      (project "caravel-breakout-wlcsp-RevA1"
+      (project "caravel-breakout-wlcsp"
         (path "/b38c65ac-2d57-46f9-9a32-ad09573ee400"
           (reference "#PWR0101") (unit 1)
@@
     (pin "1")
     (instances
-      (project "caravel-breakout-wlcsp-RevA1"
+      (project "caravel-breakout-wlcsp"
         (path "/b38c65ac-2d57-46f9-9a32-ad09573ee400"
           (reference "#PWR0103") (unit 1)
@@
     (pin "9")
     (instances
-      (project "caravel-breakout-wlcsp-RevA1"
+      (project "caravel-breakout-wlcsp"
         (path "/b38c65ac-2d57-46f9-9a32-ad09573ee400"
           (reference "CON2") (unit 1)
@@
     (pin "5")
     (instances
-      (project "caravel-breakout-wlcsp-RevA1"
+      (project "caravel-breakout-wlcsp"
         (path "/b38c65ac-2d57-46f9-9a32-ad09573ee400"
           (reference "CON3") (unit 1)

Commit message: Added fids and patch over-reliance on gnd fill for conn DRC fails
Parts:
- added FID1, FID2, FID3: Fiducial, Fiducial:Fiducial_1mm_Mask2mm, symbol Mechanical:Fiducial
Changed lines of the file:
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@@
     (stroke (width 0) (type default))
   )
-  (text "Caravel breakout (WLCSP package)" (at 118.11 20.32 0)
+  (text "Caravel breakout (WLCSP package)" (at 102.87 20.32 0)
     (effects (font (size 3 3) (thickness 0.6) bold) (justify left bottom))
   )
@@
     )
   )
+  (symbol (lib_id "Mechanical:Fiducial") (at 16.51 189.23 0) (unit 1)
+    (in_bom yes) (on_board yes) (dnp no) (fields_autoplaced)
+    (property "Reference" "FID2" (at 18.669 188.206 0)
+      (effects (font (size 1.27 1.27)) (justify left))
+    )
+    (property "Value" "Fiducial" (at 18.669 190.254 0)
+      (effects (font (size 1.27 1.27)) (justify left))
+    )
+    (property "Footprint" "Fiducial:Fiducial_1mm_Mask2mm" (at 16.51 189.23 0)
+      (effects (font (size 1.27 1.27)) hide)
+    )
+    (property "Datasheet" "~" (at 16.51 189.23 0)
+      (effects (font (size 1.27 1.27)) hide)
+    )
+    (instances
+      (project "caravel-breakout-wlcsp"
+        (path "/b38c65ac-2d57-46f9-9a32-ad09573ee400"
+          (reference "FID2") (unit 1)
+        )
+      )
+    )
+  )
+  (symbol (lib_id "Mechanical:Fiducial") (at 16.51 185.42 0) (unit 1)
+    (in_bom yes) (on_board yes) (dnp no) (fields_autoplaced)
+    (property "Reference" "FID1" (at 18.669 184.396 0)
+      (effects (font (size 1.27 1.27)) (justify left))
+    )
+    (property "Value" "Fiducial" (at 18.669 186.444 0)
+      (effects (font (size 1.27 1.27)) (justify left))
+    )
+    (property "Footprint" "Fiducial:Fiducial_1mm_Mask2mm" (at 16.51 185.42 0)
+      (effects (font (size 1.27 1.27)) hide)
+    )
+    (property "Datasheet" "~" (at 16.51 185.42 0)
+      (effects (font (size 1.27 1.27)) hide)
+    )
+    (instances
+      (project "caravel-breakout-wlcsp"
+        (path "/b38c65ac-2d57-46f9-9a32-ad09573ee400"
+          (reference "FID1") (unit 1)
+        )
+      )
+    )
+  )
   (symbol (lib_id "Connector_Generic:Conn_02x20_Odd_Even") (at 222.25 52.07 0) (unit 1)
     (in_bom yes) (on_board yes) (dnp no)
@@
         )
       )
+    )
+  )
+  (symbol (lib_id "Mechanical:Fiducial") (at 16.51 193.04 0) (unit 1)
+    (in_bom yes) (on_board yes) (dnp no) (fields_autoplaced)
+    (property "Reference" "FID3" (at 18.669 192.016 0)
+      (effects (font (size 1.27 1.27)) (justify left))
+    )
+    (property "Value" "Fiducial" (at 18.669 194.064 0)
+      (effects (font (size 1.27 1.27)) (justify left))
+    )
+    (property "Footprint" "Fiducial:Fiducial_1mm_Mask2mm" (at 16.51 193.04 0)
+      (effects (font (size 1.27 1.27)) hide)
+    )
+    (property "Datasheet" "~" (at 16.51 193.04 0)
+      (effects (font (size 1.27 1.27)) hide)
+    )
+    (instances
+      (project "caravel-breakout-wlcsp"
+        (path "/b38c65ac-2d57-46f9-9a32-ad09573ee400"
+          (reference "FID3") (unit 1)
+        )
+      )
