File: ASIC-simulator/breakout-fpga-ICE40UP5K-TT3/caravel-breakout-fpga-ICE40UP5K-TT3.kicad_pcb (KiCad board)
At the start: 2 copper layers, 45 x 52.5 mm, 173 parts, among them CON1 REF-182665-01, CON2 REF-182665-01, J3 USB4500-03-0-A_REVA, U1 AP2112K-3.3, U2 AP2112K-1.2, U3 ICE40UP5K-SG48ITR, U4 W25Q32JVSSIM, X1 20MHz

Commit message: ICE40UP5K TT3 breakout, BOM tweaks pre-PCBA first run
Parts:
- R2, R22, R23, R24, R25, R26, R27, R3, R4, R5: value R_0R_0603_JUMPER -> 0R
- R7, R8: value 0 -> 0R

Commit message: v1.2 ready for pcba
Parts:
- added C21: 0.1u, Capacitor_SMD:C_0402_1005Metric, F.Cu at (67.8, 62.1)
- added NT4: NetTie_2, NetTie:NetTie-2_SMD_Pad0.5mm, F.Cu at (90.8, 41.8)
- added NT5: NetTie_2, NetTie:NetTie-2_SMD_Pad0.5mm, F.Cu at (80.2, 39.5)
- added NT6: NetTie_2, NetTie:NetTie-2_SMD_Pad0.5mm, F.Cu at (90.4, 37.4)
- added R28: R_10k_0402, Resistor_SMD:R_0402_1005Metric, F.Cu at (66.0, 65.0)
- added R29: 1k5, Resistor_SMD:R_0603_1608Metric, F.Cu at (66.3, 60.3)
- added R30: R_10k_0402, Resistor_SMD:R_0402_1005Metric, F.Cu at (50.2, 56.9)
- added R31: 0R, Resistor_SMD:R_0603_1608Metric, F.Cu at (79.5, 22.9)
- added R32: R_100k_0402, Resistor_SMD:R_0402_1005Metric, F.Cu at (49.5, 37.4)
- added R33: R_100k_0402, Resistor_SMD:R_0402_1005Metric, F.Cu at (49.5, 46.3)
- added R34: R_100k_0402, Resistor_SMD:R_0402_1005Metric, F.Cu at (49.5, 40.0)
- added R35: R_100k_0402, Resistor_SMD:R_0402_1005Metric, F.Cu at (49.5, 34.8)
- added R36: R_100k_0402, Resistor_SMD:R_0402_1005Metric, F.Cu at (49.5, 38.7)
- added R37: R_100k_0402, Resistor_SMD:R_0402_1005Metric, F.Cu at (49.5, 45.0)
- added R38: R_100k_0402, Resistor_SMD:R_0402_1005Metric, F.Cu at (49.5, 43.8)
- added STITCH1: StitchingVia-0.3mm, flyingcarsfootprints:StitchingVia-0.3mm, F.Cu at (55.6, 64.8)
- added STITCH1: StitchingVia-0.3mm, flyingcarsfootprints:StitchingVia-0.3mm, F.Cu at (58.4, 23.6)
- added STITCH1: StitchingVia-0.3mm, flyingcarsfootprints:StitchingVia-0.3mm, F.Cu at (66.4, 47.7)
- added STITCH1: StitchingVia-0.3mm, flyingcarsfootprints:StitchingVia-0.3mm, F.Cu at (87.5, 41.2)
- added STITCH1: StitchingVia-0.3mm, flyingcarsfootprints:StitchingVia-0.3mm, F.Cu at (80.6, 66.7)
- added STITCH1: StitchingVia-0.3mm, flyingcarsfootprints:StitchingVia-0.3mm, F.Cu at (82.5, 48.9)
- added STITCH1: StitchingVia-0.3mm, flyingcarsfootprints:StitchingVia-0.3mm, F.Cu at (92.3, 46.5)
- added STITCH1: StitchingVia-0.3mm, flyingcarsfootprints:StitchingVia-0.3mm, F.Cu at (82.4, 64.1)
- added STITCH1: StitchingVia-0.3mm, flyingcarsfootprints:StitchingVia-0.3mm, F.Cu at (74.7, 60.1)
- added STITCH1: StitchingVia-0.3mm, flyingcarsfootprints:StitchingVia-0.3mm, F.Cu at (55.2, 46.0)
- added STITCH1: StitchingVia-0.3mm, flyingcarsfootprints:StitchingVia-0.3mm, F.Cu at (92.3, 42.3)
- added STITCH1: StitchingVia-0.3mm, flyingcarsfootprints:StitchingVia-0.3mm, F.Cu at (58.4, 36.4)
- added STITCH1: StitchingVia-0.3mm, flyingcarsfootprints:StitchingVia-0.3mm, F.Cu at (59.2, 41.0)
- added STITCH1: StitchingVia-0.3mm, flyingcarsfootprints:StitchingVia-0.3mm, F.Cu at (70.2, 64.8)
- added STITCH1: StitchingVia-0.3mm, flyingcarsfootprints:StitchingVia-0.3mm, F.Cu at (85.4, 53.5)
- added STITCH1: StitchingVia-0.3mm, flyingcarsfootprints:StitchingVia-0.3mm, F.Cu at (69.3, 55.8)
- added STITCH1: StitchingVia-0.3mm, flyingcarsfootprints:StitchingVia-0.3mm, F.Cu at (66.7, 55.6)
- added STITCH1: StitchingVia-0.3mm, flyingcarsfootprints:StitchingVia-0.3mm, F.Cu at (87.5, 43.7)
- added STITCH1: StitchingVia-0.3mm, flyingcarsfootprints:StitchingVia-0.3mm, F.Cu at (55.6, 60.8)
- added STITCH1: StitchingVia-0.3mm, flyingcarsfootprints:StitchingVia-0.3mm, F.Cu at (63.8, 61.9)
- added STITCH1: StitchingVia-0.3mm, flyingcarsfootprints:StitchingVia-0.3mm, F.Cu at (78.5, 47.1)
- added STITCH1: StitchingVia-0.3mm, flyingcarsfootprints:StitchingVia-0.3mm, F.Cu at (56.0, 31.4)
- added STITCH1: StitchingVia-0.3mm, flyingcarsfootprints:StitchingVia-0.3mm, F.Cu at (58.4, 33.8)
- added STITCH1: StitchingVia-0.3mm, flyingcarsfootprints:StitchingVia-0.3mm, F.Cu at (79.5, 61.1)
- added STITCH1: StitchingVia-0.3mm, flyingcarsfootprints:StitchingVia-0.3mm, F.Cu at (68.9, 62.6)
- added STITCH1: StitchingVia-0.3mm, flyingcarsfootprints:StitchingVia-0.3mm, F.Cu at (61.2, 27.6)
- added STITCH1: StitchingVia-0.3mm, flyingcarsfootprints:StitchingVia-0.3mm, F.Cu at (89.6, 41.2)
- added STITCH1: StitchingVia-0.3mm, flyingcarsfootprints:StitchingVia-0.3mm, F.Cu at (75.3, 65.4)
- added STITCH1: StitchingVia-0.3mm, flyingcarsfootprints:StitchingVia-0.3mm, F.Cu at (82.5, 46.4)
- added STITCH1: StitchingVia-0.3mm, flyingcarsfootprints:StitchingVia-0.3mm, F.Cu at (55.6, 41.0)
- added STITCH1: StitchingVia-0.3mm, flyingcarsfootprints:StitchingVia-0.3mm, F.Cu at (85.4, 61.1)
- added STITCH1: StitchingVia-0.3mm, flyingcarsfootprints:StitchingVia-0.3mm, F.Cu at (77.7, 63.6)
- added STITCH1: StitchingVia-0.3mm, flyingcarsfootprints:StitchingVia-0.3mm, F.Cu at (61.7, 63.8)
- added STITCH1: StitchingVia-0.3mm, flyingcarsfootprints:StitchingVia-0.3mm, F.Cu at (58.3, 26.2)
- added STITCH1: StitchingVia-0.3mm, flyingcarsfootprints:StitchingVia-0.3mm, F.Cu at (85.4, 58.9)
- added STITCH1: StitchingVia-0.3mm, flyingcarsfootprints:StitchingVia-0.3mm, F.Cu at (63.9, 57.6)
- added STITCH1: StitchingVia-0.3mm, flyingcarsfootprints:StitchingVia-0.3mm, F.Cu at (56.2, 51.3)
- added STITCH1: StitchingVia-0.3mm, flyingcarsfootprints:StitchingVia-0.3mm, F.Cu at (82.5, 41.2)
- added STITCH1: StitchingVia-0.3mm, flyingcarsfootprints:StitchingVia-0.3mm, F.Cu at (85.4, 50.8)
- added STITCH1: StitchingVia-0.3mm, flyingcarsfootprints:StitchingVia-0.3mm, F.Cu at (77.5, 54.8)
- added STITCH1: StitchingVia-0.3mm, flyingcarsfootprints:StitchingVia-0.3mm, F.Cu at (58.4, 30.8)
- added STITCH1: StitchingVia-0.3mm, flyingcarsfootprints:StitchingVia-0.3mm, F.Cu at (82.5, 43.7)
- added STITCH24: StitchingVia-0.3mm, flyingcarsfootprints:StitchingVia-0.3mm, F.Cu at (66.5, 66.0)
- added STITCH32: StitchingVia-0.3mm, flyingcarsfootprints:StitchingVia-0.3mm, F.Cu at (79.9, 25.0)
- added SW1: 434121025816, TinyTapeout:434121025816, F.Cu at (62.3, 65.0)
- added kibuzzard-6288F08E: G***, kibuzzard-6288F08E, F.Cu at (91.0, 42.4)
- R25, R26: value 0R -> R_10k_0402; footprint Resistor_SMD:R_0603_1608Metric -> Resistor_SMD:R_0402_1005Metric
- R27: value 0R -> R_100k_0402; footprint Resistor_SMD:R_0603_1608Metric -> Resistor_SMD:R_0402_1005Metric
- moved R26 47.2 mm to (50.3, 61.2), turned to 180 degrees
- moved R27 31.6 mm to (49.5, 36.1), turned to 180 degrees
- moved R24 30.7 mm to (74.9, 67.9), turned to 90 degrees
- moved R25 12.7 mm to (73.2, 50.8), turned to 0 degrees
- moved R11 2.34 mm to (67.8, 64.3), turned to 90 degrees
- moved STITCH4 2.24 mm to (49.0, 33.8)
- moved STITCH1 1.90 mm to (71.5, 57.7)
- moved D4 1.77 mm to (66.1, 62.8), turned to -90 degrees
- moved STITCH1 1.44 mm to (74.0, 48.9)
- moved STITCH6 1.40 mm to (49.0, 47.6)
- moved R21 1.32 mm to (72.0, 53.9)
- moved STITCH3 1.16 mm to (49.0, 29.8)
- moved STITCH1 1.00 mm to (66.4, 40.2)
- moved STITCH1 0.99 mm to (79.4, 57.1)
- moved STITCH5 0.80 mm to (49.0, 41.9)
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Connections:
- C8 pad 1: +1V8 -> +3V3
- CON1 pad 38: xclk -> Net-(CON1-Pin_38)
- R24 pad 1: Caravel_SCK -> mprj_io[3]_CSB
- R24 pad 2: /FT_SCK -> /FT_SSn
- R25 pad 1: Caravel_D1 -> mprj_io[13]
- R25 pad 2: /FLASH_MOSI -> GND
- R26 pad 1: Caravel_D0 -> mprj_io[12]
- R26 pad 2: /FLASH_MISO -> GND
- R27 pad 1: +3V3 -> mprj_io[27]
- R27 pad 2: +1V8 -> GND
- U2 pad 1: +1V8 -> +3V3
- U2 pad 3: +1V8 -> +3V3
- U3 pad 9: mprj_io[15] -> BOOT
Routing:
- net mprj_io[3]_CSB: track 26.9 -> 59.7 mm, vias 2 -> 4
- net GND: track 55.9 -> 86.6 mm, vias 35 -> 43
- net mprj_io[15]: track 19.5 -> 0.00 mm
- net BOOT: track 0.00 -> 17.6 mm, vias 0 -> 2
- net +1V8: track 53.6 -> 41.7 mm
- net Net-(R28-Pad2): track 0.00 -> 10.2 mm, vias 0 -> 2
- net mprj_io[27]: track 12.8 -> 21.8 mm
- net mprj_io[21]: track 11.8 -> 20.7 mm
- net mprj_io[25]: track 30.7 -> 39.7 mm
- net mprj_io[23]: track 25.5 -> 34.5 mm
- net +3V3: track 152.5 -> 160.3 mm, vias 17 -> 16
- net Net-(C18-Pad1): track 3.40 -> 7.40 mm
- net Net-(CON1-Pin_38): track 0.00 -> 3.07 mm
- net mprj_io[26]: track 18.5 -> 21.3 mm
- net mprj_io[24]: track 16.6 -> 19.4 mm
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Other:
- board text added: "(C) 2024 Pat Deegan"
- board text added: "BOOT"
- board text added: "CD1"
- board text added: "CSCK"
- board text added: "ICE40UP5K/TT3 variant, v1.2"
- board text added: "TT3 v1.2"
- board text added: "in0"
- board text added: "in1/io22"
- board text added: "in2"
- board text added: "in3/io24"
- board text added: "in4"
- board text added: "in5/io26"
- board text added: "in6"
- board text added: "in7/io28"
- board text added: "io03 HKcsb"
- board text added: "out0"
- board text added: "out1"
- board text added: "out1/io30"
- board text added: "out2"
- board text added: "out3"
- board text added: "out3/io32"
- board text added: "out4"
- board text added: "out5"
- board text added: "out5/io34"
- board text added: "out6/io35"
- board text added: "out7"
- board text added: "out7/io36"
- board text added: "sel0"
- board text added: "sel2"
- board text added: "sl0/io12"
- board text added: "sl1"
- board text added: "sl2/io14"
- board text added: "v1.2"
- board text removed: "(C) 2023 Pat Deegan"
- board text removed: "Csck"
- board text removed: "ICE40UP5K/TT3 variant, v1.0"
- board text removed: "TT3 v1.0"
- board text removed: "io03 csb"
- board text removed: "io12"
- board text removed: "io13"
- board text removed: "io14"
- board text removed: "io21"
- board text removed: "io22"
- board text removed: "io23"
- board text removed: "io24"
- board text removed: "io25"
- board text removed: "io26"
- board text removed: "io27"
- board text removed: "io28"
- board text removed: "io29"
- board text removed: "io30"
- board text removed: "io31"
- board text removed: "io32"
- board text removed: "io33"
- board text removed: "io34"
- board text removed: "io35"
- board text removed: "io36"
- board text removed: "tinytapeout.com"
- board text removed: "v1.0"
