File: breakout-qfn/caravel-breakout-qfn.kicad_sch (KiCad schematic)
At the start: 13 parts, among them CON1 REF-182665-01, CON2 REF-182665-01, U1 Caravel_QFN_TT4

Commit message: v3.2 moved to bottom side pin headers
Parts:
- added FID1, FID2, FID3: Fiducial, Fiducial:Fiducial_1mm_Mask2mm, symbol Mechanical:Fiducial
- CON1: value REF-182665-01 -> ~; footprint BreakoutCommon:FH-00339 -> TinyTapeout:FH-00148_PinSocket_2x20_P2.54mm; Characteristics (none) -> 2x20 100 mil Receptacle SMT; DigikeyPN (none) -> S5690-ND; JLC (none) -> C2685092; MPN FH-00339 -> NPTC202KFMS-RC; MPN_ALT REF-182665-01 (or Harwin M20-7812045) -> FH-00148
- CON2: value REF-182665-01 -> ~; footprint BreakoutCommon:FH-00339 -> TinyTapeout:FH-00148_PinSocket_2x20_P2.54mm; DigikeyPN (none) -> S5690-ND; JLC (none) -> C2685092; MPN FH-00339 -> NPTC202KFMS-RC; MPN_ALT REF-182665-01 (or Harwin M20-7812045) -> FH-00148
Other:
- note added: "CON1, CON2: Place on bottom"
